File: mic_amp.sch (KiCad schematic (older format))
At the start: 25 parts

Commit message: filling wanted :)
Parts:
- removed HOLE1: HOLE_METALLED, PCB:Hole3_5_out6mm, symbol HOLE_METALLED
Connections:
- wire segments 70 -> 69
Changed lines of the file:
@@
 MICIN
 Wire Wire Line
-	3900 3600 4150 3600
-Wire Wire Line
-	4150 3600 4150 2500
+	4150 3600 3900 3600
+Wire Wire Line
+	4150 2500 4150 3600
 Wire Wire Line
 	4150 2500 4450 2500
@@
 Wire Wire Line
 	7750 5250 7900 5250
-$Comp
-L HOLE_METALLED HOLE1
-U 1 1 56235597
-P 9750 5300
-F 0 "HOLE1" H 9250 5250 60  0000 C CNN
-F 1 "HOLE_METALLED" H 9200 5350 60  0000 C CNN
-F 2 "PCB:Hole3_5_out6mm" H 9750 5300 60  0001 C CNN
-F 3 "" H 9750 5300 60  0000 C CNN
-	1    9750 5300
-	1    0    0    -1
-$EndComp
-$Comp
-L GND #PWR028
-U 1 1 56235764
-P 10200 5300
-F 0 "#PWR028" H 10290 5280 30  0001 C CNN
-F 1 "GND" H 10200 5220 30  0001 C CNN
-F 2 "" H 10200 5300 60  0000 C CNN
-F 3 "" H 10200 5300 60  0000 C CNN
-	1    10200 5300
-	0    1    1    0
-$EndComp
-Wire Wire Line
-	10050 5300 10200 5300
 Wire Wire Line
 	8400 3300 8200 3300

Commit message: With 3v battery
Parts:
- removed C1: 10n, Capacitors:CAP_0603, symbol C
- removed C2: 1u, Capacitors:CAP_0603, symbol C
- removed DA1: NCP662SQ, SOT:SC82AB, symbol NCP662SQ
- removed F1, F2: Fuse0R, Resistors:RES_0603_SOLDERFUSE, symbol Fuse0R
- removed R1: 1M, Resistors:RES_0603, symbol R
- removed XL1: USB_MINI_B, Connectors:USBmicro_MOLEX_WM17142, symbol USB_MINI_B
- removed XL2: CONN_AUDIO_SIMPLE, Connectors:AUDIO_CKX3_5_30, symbol CONN_AUDIO_SIMPLE
- added B1: BAT, Installation:BAT_HOLDER_BHX1-2032-SM, symbol BAT
- added C8, C9: 1u, Capacitors:CAP_0603, symbol C
- added D3: BAT54WS, Diodes:SOD323, symbol D_Shottky
- added HOLE1, HOLE2: HOLE_METALLED, PCB:Hole3d3_out5d5mm, symbol HOLE_METALLED
- added Q1: IRLML9303, SOT:SOT23-3, symbol MOSFET_P_3LEAD
- added Q2: BC848, SOT:SOT23-3, symbol NPN
- added R2: 0R, Resistors:RES_0603, symbol R
- added R5: 20k, Resistors:RES_0603, symbol R
- added R8: 2k, Resistors:RES_0603, symbol R
- added SW1: SWITCH, BtnsSwitches:SW_SS-1P2T, symbol SWITCH
- added XL1, XL3: CONN_2, Connectors:PLS-2, symbol CONN_2
- C5: renamed from C6; value 0.1u -> 10u
- C6: renamed from C8; value 1u -> 0.1u
- R3: value 150k -> DNM; Price (none) -> 0.5; SolderPoints (none) -> 2
- R4: value 100k -> 2k; Price (none) -> 0.5; SolderPoints (none) -> 2
- R6: value 1k -> 2k; Price (none) -> 0.5; SolderPoints (none) -> 2
- renumbered C4 to C1, C3 to C2, C5 to C3, C7 to C4, C9 to C7, D2 to D1, D1 to D2, F3 to F1, R2 to R1, R5 to R7, XL3 to XL2
Connections:
- net labels added: BAT_IN
- wire segments 69 -> 75
- no-connect marks 3 -> 2
Other:
- note added: "AGC disabled"
- note added: "Attack/release ratio:\nNot soldered: 1:4000"
- note added: "Gain select:\nGAIN = GND: gain = 50dB\nGAIN not connected: gain = 60dB"
- note removed: "Attack/release ratio:\nSoldered: 1:500\nNot soldered: 1:4000"
- note removed: "Connect TH to MICBIAS\nto disable the AGC."
- note removed: "Gain select:\nGAIN = Vdd: gain = 40dB\nGAIN = GND: gain = 50dB\nGAIN not connected: gain = 60dB"
- moved on the sheet: C1, C2, C3, C4, C5, C6, C7, D1, D2, F1, R1

Commit message: 2xAAA sch
Parts:
- removed B1: BAT, Installation:BAT_HOLDER_BHX1-2032-SM, symbol BAT
- removed C5: 10u, Capacitors:CAP_0603, symbol C
- removed D3: BAT54WS, Diodes:SOD323, symbol D_Shottky
- removed Q1: IRLML9303, SOT:SOT23-3, symbol MOSFET_P_3LEAD
- removed Q2: BC848, SOT:SOT23-3, symbol NPN
- removed R5: 20k, Resistors:RES_0603, symbol R
- removed R7: 20k, Resistors:VAR_PTV09A-4, symbol RVar
- removed SW1: SWITCH, BtnsSwitches:SW_SS-1P2T, symbol SWITCH
- removed XL2: CONN_AUDIO_SIMPLE, Connectors:AUDIO_CKX3_5_30, symbol CONN_AUDIO_SIMPLE
- removed XL3: CONN_2, Connectors:PLS-2, symbol CONN_2
- added B1: BAT_HOLDER, Installation:BATTERY_AAA_X2, symbol BAT_HOLDER
- added C10, C6: 1u, Capacitors:CAP_0603, symbol C
- added DA1: TPA6211, QFN_DFN:DRB8, symbol TPA6211
- added R5: RVarWSw, Resistors:RVar_SP3, symbol RVarWSw
- added R7: 10k, Resistors:RES_0603, symbol R
- added R8: 0R, Resistors:RES_0603, symbol R
- added XL2: AudioJackSimple, Connectors:AUDIO_CKX3_5_30, symbol AudioJackSimple
- added XL3: AudioJackSimple_x4, Connectors:Audio_ST013, symbol AudioJackSimple_x4
- R6: value 2k -> 10k; Price 0.5 -> (none); SolderPoints 2 -> (none)
- renumbered C6 to C5, R8 to R9
Connections:
- net labels added: +3.3V, +BATT, Output
- net labels removed: BAT_IN, VDD
- wire segments 75 -> 81
- no-connect marks 2 -> 4
Other:
- note added: "2xAAA"
- note added: "Headphones"
- note added: "Power"
- moved on the sheet: D1, HOLE1, HOLE2, R4, R9

Commit message: + Pcb sent to manufacturing
Parts:
- removed B1: BAT_HOLDER, Installation:BATTERY_AAA_X2, symbol BAT_HOLDER
- added B1: BAT, Installation:BATTERY_AAA_X1, symbol BAT
- added C11, C13, C14: 10u, Capacitors:CAP_0603, symbol C
- added C12: 0.1u, Capacitors:CAP_0603, symbol C
- added D3: BAT54WS, Diodes:SOD323, symbol D_Shottky
- added DA2: NCP140x, SOT:SOT23-5, symbol NCP140x
- added HOLE3, HOLE4: HOLE_METALLED, PCB:Hole3d3_out5d5mm, symbol HOLE_METALLED
- added L1: 22uH, Inductors:IND_1210_LQH32C, symbol L
- added L2: BLM15AG102, Inductors:IND_0402, symbol L
- R5: footprint Resistors:RVar_SP3 -> Resistors:RVar_SP3_R
Connections:
- net +3.3V: now also C14.2, L2.1; no longer R5.5
- net +BATT: now also R5.5, C11.2, C12.2, L1.2; no longer R5.4
- net GND: now also XL2.H, B1.C, C11.1, C12.1, C13.1, C14.1, DA2.4 (GND), HOLE3.H, HOLE4.H
- new net 3v3unfil: C13.2, D3.C, DA2.1 (CE), DA2.2 (OUT), L2.2
- new net BAT_IN: B1.A, R5.4
- new net Lout: D3.A, DA2.5 (LX), L1.1
- no-connect marks 4 -> 3
Other:
- note added: "1xAAA"
- note added: "Power +3V3"
- note removed: "2xAAA"
- moved on the sheet: HOLE1, HOLE2

Commit message: Proceeding with sch
Parts:
- removed R2: 0R, Resistors:RES_0603, symbol R
- removed R3: DNM, Resistors:RES_0603, symbol R
- removed R5: RVarWSw, Resistors:RVar_SP3_R, symbol RVarWSw
- added C? (x2): 0.1u, Capacitors:CAP_0603, symbol C
- added C?: 1u, Capacitors:CAP_0603, symbol C
- added C?: 10n, Capacitors:CAP_0603, symbol C
- added DD?: STM32F030F6Px, SO_DIL_TSSOP:TSSOP20, symbol STM32F030F6Px
- added DD?: MC4011, QFN_DFN:DFN8_2x3, symbol MC4011
- added L?: BLM15AG102, Inductors:IND_0402, symbol L
- added SW? (x2): IT-1198E, BtnsSwitches:BTN_IT1198, symbol BUTTON_H
- added XL?: CONN_3, Connectors:PLS-3, symbol CONN_3
- added XL?: ST_SWD, Connectors:PLS-4, symbol ST_SWD
- R4: value 2k -> 1k
- R8: value 0R -> 15k
Connections:
- net +3.3V: now also C?.1, DD?.1 (Vdd); no longer R4.1
- net +BATT: now also DD?.8 (ADC2/TX1/PA2), XL?.1 (Vdd)
- net 3v3unfil: now also C?.1, DD?.16 (VDD), L?.2
- net GND: now also C?.2, C?.2, C?.2, C?.2, DD?.15 (VSS), DD?.2 (Vss), DD?.6 (B), DD?.PAD, SW?.1, SW?.1, SW?.H, SW?.H, XL?.1 (P1), XL?.3 (GND)
- net MICIN: now also C1.2
- net W: now reaches C6.1
- net W: now also DD?.4 (W)
- net Output renamed MicAmpOut
- net MicAmpOut: now also DD?.3 (A)
- new net: DD?.12 (ADC6/MISO1/T3C1/T16C1/PA6), R4.1
- new net: C?.1, C?.1, DD?.5 (VDDA), L?.1
- new net: DD?.6 (ADC0/WKUP1/PA0), SW?.2
- new net: DD?.7 (ADC1/PA1), SW?.2
- new net CS: DD?.11 (ADC5/SCK1/PA5), DD?.5 (~CS)
- new net SWCLK: DD?.20 (SWCLK/PA14), XL?.2 (SWCLK)
- new net SWDIO: DD?.19 (IR_OUT/SWDIO/PA13), XL?.4 (SWDIO)
- new net UART_RX: DD?.18 (RX1/SDA1/T1C3/PA10), XL?.3
- new net UART_TX: DD?.17 (TX1/SCL1/T1C2/PA9), XL?.2 (PM)
- new net UD: DD?.10 (ADC4/T14C1/PA4), DD?.8 (U/~D)
- no-connect marks 3 -> 10
Other:
- note added: "Battery \nmeasurement"
- note added: "Debug port"
- note added: "Programming"
- note added: "Smartphone"
- moved on the sheet: B1, C1, C11, C12, C13, C14, C2, C3, C4, C5, C9, D1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

Commit message: + mic amp 2.1 pcb ready
Parts:
- removed XL?: CONN_3, Connectors:PLS-3, symbol CONN_3
- removed XL?: ST_SWD, Connectors:PLS-4, symbol ST_SWD
- added C19: 10u, Capacitors:CAP_0603, symbol C
- added C20: 0.1u, Capacitors:CAP_0603, symbol C
- added D4: LED, LEDs:LED_0603, symbol LED
- added R2: 10k, Resistors:RES_0603, symbol R
- added R3: 390k, Resistors:RES_0603, symbol R
- added R5: 1k, Resistors:RES_0603, symbol R
- added SW3: IT-1198E, BtnsSwitches:BTN_IT1198, symbol BUTTON_H
- added XL4: CONN_6, Connectors:PLS-6, symbol CONN_6
- D1: footprint LEDs:LED_Through-Hole-3mm -> LEDs:LED_0603
- D3: value BAT54WS -> PMEG3010; Price 2.5 -> 5; URL https://www.terraelectronica.ru/catalog_info.php?CODE=182655 -> (none)
- HOLE1, HOLE2, HOLE3, HOLE4: footprint PCB:Hole3d3_out5d5mm -> PCB:Hole2d4_out4d5mm
- XL3: footprint Connectors:Audio_ST013 -> Connectors:Audio_ST511D01TR; PN ST-013 -> ST-511D-01-TR; Price (none) -> 42; SolderPoints (none) -> 5; URL http://www.chipdip.ru/product/st-013/ -> http://www.eltech.spb.ru/item/st_511d_01_tr
- gave numbers to parts that had none: 9
Connections:
- net BAT_IN is gone; now on net +BATT: B1.A
- net +BATT: now also R2.1; no longer DD1.8 (ADC2/TX1/PA2)
- net 3v3unfil: now also C20.2, XL4.1; no longer DA2.1 (CE)
- net GND: now also C19.1, C20.1, D4.C, R3.2, SW3.H, XL4.3
- net SWCLK: now also XL4.2
- net SWDIO: now also XL4.4
- net UART_RX: now also XL4.6
- net UART_TX: now also XL4.5
- net at DD1.13 (ADC7/MOSI1/T3C2/T14C1/T1C1N/T17C1/PA7): now also R5.1
- net BTN_CHCK: now reaches DD1.9 (ADC3/RX1/PA3)
- net BTN_CHCK: now also R2.2, SW3.2
- new net: D4.A, R5.2
- new net PWR_EN: C19.2, DA2.1 (CE), DD1.8 (ADC2/TX1/PA2), R3.1, SW3.1
- no-connect marks 10 -> 8
Other:
- note added: "1) Off, btn released => PWR_EN == 0V\n2) Off, btn pressed => PWR_EN == 1.5V, BTN_CHCK == 1.5V\n3) MCU sets PWR_EN = 3.3V\n4) On, btn released => PWR_EN == 3.3V by MCU, BTN_CHCK == 1.5V\n5) On, btn pressed => PWR_EN == 3.3V by MCU, BTN_CHCK == 3.3V \n6) MCU thus detects btn press and waits btn release (BTN_CHCK == 1.5V)\n7) MCU sets PWR_EN = 0 to switch system off"
- note added: "Programming & debug"
- note removed: "Battery \nmeasurement"
- note removed: "Debug port"
- note removed: "Programming"
- moved on the sheet: B1, C11, C12, C13, C14, C15, C16, C17, D1, D3, DA2, DD1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
